Commit message: go2 model visible in rviz

File: go2_navigation/urdf/go2_navigation.urdf.xacro (robot description, xacro)
@@ -10,5 +10,5 @@
       <origin xyz="0 0 0" rpy="0 0 0" />
       <geometry>
-        <mesh filename="package://go2_navigation/meshes/dae/base.dae" />
+        <mesh filename="package://go2_navigation/meshes/base.dae" />
       </geometry>
       <material name="深色橡胶_001-effect"><color rgba="0.6717055 0.6924257 0.7742702 1" /></material><material name="白色logo_001-effect"><color rgba="1 1 1 1" /></material><material name="黑色贴纸_007-effect"><color rgba="0.009018 0.009018 0.009018 1" /></material><material name="黑色金属_007-effect"><color rgba="0.01341 0.01341 0.01341 1" /></material><material name="黑色塑料_003-effect"><color rgba="0.023455 0.023455 0.023455 1" /></material></visual>
@@ -67,5 +67,5 @@
       <origin xyz="0 0 0" rpy="0 0 0" />
       <geometry>
-        <mesh filename="package://go2_navigation/meshes/dae/hip.dae" />
+        <mesh filename="package://go2_navigation/meshes/hip.dae" />
       </geometry>
       <material name="深色橡胶_001-effect"><color rgba="0.6717055 0.6924257 0.7742702 1" /></material><material name="Material-effect"><color rgba="0.9 0.95 0.95 1" /></material></visual>
@@ -105,5 +105,5 @@
       <origin xyz="0 0 0" rpy="0 0 0" />
       <geometry>
-        <mesh filename="package://go2_navigation/meshes/dae/thigh.dae" />
+        <mesh filename="package://go2_navigation/meshes/thigh.dae" />
       </geometry>
       <material name="深色橡胶_003-effect"><color rgba="0.6717055 0.6924257 0.7742702 1" /></material><material name="Material_009-effect"><color rgba="0.9 0.95 0.95 1" /></material></visual>
@@ -143,5 +143,5 @@
       <origin xyz="0 0 0" rpy="0 0 0" />
       <geometry>
-        <mesh filename="package://go2_navigation/meshes/dae/calf.dae" />
+        <mesh filename="package://go2_navigation/meshes/calf.dae" />
       </geometry>
       <material name="黑色足端_005-effect"><color rgba="0 0 0 1" /></material><material name="深色橡胶_005-effect"><color rgba="0.6717055 0.6924257 0.7742702 1" /></material></visual>
@@ -209,5 +209,5 @@
       <origin xyz="0 0 0" rpy="0 0 0" />
       <geometry>
-        <mesh filename="package://go2_navigation/meshes/dae/foot.dae" />
+        <mesh filename="package://go2_navigation/meshes/foot.dae" />
       </geometry>
       <material name="黑色足端_007-effect"><color rgba="0 0 0 1" /></material></visual>
@@ -234,5 +234,5 @@
       <origin xyz="0 0 0" rpy="3.1415 0 0" />
       <geometry>
-        <mesh filename="package://go2_navigation/meshes/dae/hip.dae" />
+        <mesh filename="package://go2_navigation/meshes/hip.dae" />
       </geometry>
       <material name="深色橡胶_001-effect"><color rgba="0.6717055 0.6924257 0.7742702 1" /></material><material name="Material-effect"><color rgba="0.9 0.95 0.95 1" /></material></visual>
@@ -272,5 +272,5 @@
       <origin xyz="0 0 0" rpy="0 0 0" />
       <geometry>
-        <mesh filename="package://go2_navigation/meshes/dae/thigh_mirror.dae" />
+        <mesh filename="package://go2_navigation/meshes/thigh_mirror.dae" />
       </geometry>
       <material name="深色橡胶_012-effect"><color rgba="0.6717055 0.6924257 0.7742702 1" /></material><material name="Material_011-effect"><color rgba="0.9 0.95 0.95 1" /></material></visual>
@@ -310,5 +310,5 @@
       <origin xyz="0 0 0" rpy="0 0 0" />
       <geometry>
-        <mesh filename="package://go2_navigation/meshes/dae/calf_mirror.dae" />
+        <mesh filename="package://go2_navigation/meshes/calf_mirror.dae" />
       </geometry>
       <material name="黑色足端_006-effect"><color rgba="0 0 0 1" /></material><material name="深色橡胶_007-effect"><color rgba="0.6717055 0.6924257 0.7742702 1" /></material></visual>
@@ -376,5 +376,5 @@
       <origin xyz="0 0 0" rpy="0 0 0" />
       <geometry>
-        <mesh filename="package://go2_navigation/meshes/dae/foot.dae" />
+        <mesh filename="package://go2_navigation/meshes/foot.dae" />
       </geometry>
       <material name="黑色足端_007-effect"><color rgba="0 0 0 1" /></material></visual>
@@ -401,5 +401,5 @@
       <origin xyz="0 0 0" rpy="0 3.1415 0" />
       <geometry>
-        <mesh filename="package://go2_navigation/meshes/dae/hip.dae" />
+        <mesh filename="package://go2_navigation/meshes/hip.dae" />
       </geometry>
       <material name="深色橡胶_001-effect"><color rgba="0.6717055 0.6924257 0.7742702 1" /></material><material name="Material-effect"><color rgba="0.9 0.95 0.95 1" /></material></visual>
@@ -439,5 +439,5 @@
       <origin xyz="0 0 0" rpy="0 0 0" />
       <geometry>
-        <mesh filename="package://go2_navigation/meshes/dae/thigh.dae" />
+        <mesh filename="package://go2_navigation/meshes/thigh.dae" />
       </geometry>
       <material name="深色橡胶_003-effect"><color rgba="0.6717055 0.6924257 0.7742702 1" /></material><material name="Material_009-effect"><color rgba="0.9 0.95 0.95 1" /></material></visual>
@@ -477,5 +477,5 @@
       <origin xyz="0 0 0" rpy="0 0 0" />
       <geometry>
-        <mesh filename="package://go2_navigation/meshes/dae/calf.dae" />
+        <mesh filename="package://go2_navigation/meshes/calf.dae" />
       </geometry>
       <material name="黑色足端_005-effect"><color rgba="0 0 0 1" /></material><material name="深色橡胶_005-effect"><color rgba="0.6717055 0.6924257 0.7742702 1" /></material></visual>
@@ -543,5 +543,5 @@
       <origin xyz="0 0 0" rpy="0 0 0" />
       <geometry>
-        <mesh filename="package://go2_navigation/meshes/dae/foot.dae" />
+        <mesh filename="package://go2_navigation/meshes/foot.dae" />
       </geometry>
       <material name="黑色足端_007-effect"><color rgba="0 0 0 1" /></material></visual>
@@ -568,5 +568,5 @@
       <origin xyz="0 0 0" rpy="3.1415 3.1415 0" />
       <geometry>
-        <mesh filename="package://go2_navigation/meshes/dae/hip.dae" />
+        <mesh filename="package://go2_navigation/meshes/hip.dae" />
       </geometry>
       <material name="深色橡胶_001-effect"><color rgba="0.6717055 0.6924257 0.7742702 1" /></material><material name="Material-effect"><color rgba="0.9 0.95 0.95 1" /></material></visual>
@@ -606,5 +606,5 @@
       <origin xyz="0 0 0" rpy="0 0 0" />
       <geometry>
-        <mesh filename="package://go2_navigation/meshes/dae/thigh_mirror.dae" />
+        <mesh filename="package://go2_navigation/meshes/thigh_mirror.dae" />
       </geometry>
       <material name="深色橡胶_012-effect"><color rgba="0.6717055 0.6924257 0.7742702 1" /></material><material name="Material_011-effect"><color rgba="0.9 0.95 0.95 1" /></material></visual>
@@ -644,5 +644,5 @@
       <origin xyz="0 0 0" rpy="0 0 0" />
       <geometry>
-        <mesh filename="package://go2_navigation/meshes/dae/calf_mirror.dae" />
+        <mesh filename="package://go2_navigation/meshes/calf_mirror.dae" />
       </geometry>
       <material name="黑色足端_006-effect"><color rgba="0 0 0 1" /></material><material name="深色橡胶_007-effect"><color rgba="0.6717055 0.6924257 0.7742702 1" /></material></visual>
@@ -710,5 +710,5 @@
       <origin xyz="0 0 0" rpy="0 0 0" />
       <geometry>
-        <mesh filename="package://go2_navigation/meshes/dae/foot.dae" />
+        <mesh filename="package://go2_navigation/meshes/foot.dae" />
       </geometry>
       <material name="黑色足端_007-effect"><color rgba="0 0 0 1" /></material></visual>

Commit message: build tf tree

File: go2_navigation/urdf/go2_navigation.urdf.xacro (robot description, xacro)
@@ -1,5 +1,5 @@
 <?xml version='1.0' encoding='utf-8'?>
 <robot name="go2_navigation">
-  <link name="base">
+  <link name="base_link">
     <inertial>
       <origin xyz="0.021112 0 -0.005366" rpy="0 0 0" />
@@ -10,5 +10,5 @@
       <origin xyz="0 0 0" rpy="0 0 0" />
       <geometry>
-        <mesh filename="package://go2_navigation/meshes/base.dae" />
+        <mesh filename="package://go2_navigation/meshes/base_link.dae" />
       </geometry>
       <material name="深色橡胶_001-effect"><color rgba="0.6717055 0.6924257 0.7742702 1" /></material><material name="白色logo_001-effect"><color rgba="1 1 1 1" /></material><material name="黑色贴纸_007-effect"><color rgba="0.009018 0.009018 0.009018 1" /></material><material name="黑色金属_007-effect"><color rgba="0.01341 0.01341 0.01341 1" /></material><material name="黑色塑料_003-effect"><color rgba="0.023455 0.023455 0.023455 1" /></material></visual>
@@ -35,5 +35,5 @@
   <joint name="Head_upper_joint" type="fixed" dont_collapse="true">
     <origin xyz="0.285 0 0.01" rpy="0 0 0" />
-    <parent link="base" />
+    <parent link="base_link" />
     <child link="Head_upper" />
     <axis xyz="0 0 0" />
@@ -79,5 +79,5 @@
   <joint name="FL_hip_joint" type="revolute">
     <origin xyz="0.1934 0.0465 0" rpy="0 0 0" />
-    <parent link="base" />
+    <parent link="base_link" />
     <child link="FL_hip" />
     <axis xyz="1 0 0" />
@@ -93,5 +93,5 @@
   <joint name="FL_hip_rotor_joint" type="fixed">
     <origin rpy="0 0 0" xyz="0.11215 0.04675 0" />
-    <parent link="base" />
+    <parent link="base_link" />
     <child link="FL_hip_rotor" />
   </joint>
@@ -246,5 +246,5 @@
   <joint name="FR_hip_joint" type="revolute">
     <origin xyz="0.1934 -0.0465 0" rpy="0 0 0" />
-    <parent link="base" />
+    <parent link="base_link" />
     <child link="FR_hip" />
     <axis xyz="1 0 0" />
@@ -260,5 +260,5 @@
   <joint name="FR_hip_rotor_joint" type="fixed">
     <origin rpy="0 0 0" xyz="0.11215 -0.04675 0" />
-    <parent link="base" />
+    <parent link="base_link" />
     <child link="FR_hip_rotor" />
   </joint>
@@ -413,5 +413,5 @@
   <joint name="RL_hip_joint" type="revolute">
     <origin xyz="-0.1934 0.0465 0" rpy="0 0 0" />
-    <parent link="base" />
+    <parent link="base_link" />
     <child link="RL_hip" />
     <axis xyz="1 0 0" />
@@ -427,5 +427,5 @@
   <joint name="RL_hip_rotor_joint" type="fixed">
     <origin rpy="0 0 0" xyz="-0.11215 0.04675 0" />
-    <parent link="base" />
+    <parent link="base_link" />
     <child link="RL_hip_rotor" />
   </joint>
@@ -580,5 +580,5 @@
   <joint name="RR_hip_joint" type="revolute">
     <origin xyz="-0.1934 -0.0465 0" rpy="0 0 0" />
-    <parent link="base" />
+    <parent link="base_link" />
     <child link="RR_hip" />
     <axis xyz="1 0 0" />
@@ -594,5 +594,5 @@
   <joint name="RR_hip_rotor_joint" type="fixed">
     <origin rpy="0 0 0" xyz="-0.11215 -0.04675 0" />
-    <parent link="base" />
+    <parent link="base_link" />
     <child link="RR_hip_rotor" />
   </joint>
@@ -735,5 +735,5 @@
   <joint name="imu_joint" type="fixed">
     <origin xyz="-0.02557 0 0.04232" rpy="0 0 0" />
-    <parent link="base" />
+    <parent link="base_link" />
     <child link="imu" />
     <axis xyz="0 0 0" />
@@ -748,5 +748,5 @@
   <joint name="radar_joint" type="fixed">
     <origin xyz="0.28945 0 -0.046825" rpy="0 2.8782 0" />
-    <parent link="base" />
+    <parent link="base_link" />
     <child link="radar" />
     <axis xyz="0 0 0" />
@@ -754,5 +754,5 @@
   <joint name="front_camera_joint" type="fixed">
     <origin rpy="0 0 0" xyz="0.32715 -0.00003 0.04297" />
-      <parent link="base" />
+      <parent link="base_link" />
       <child link="front_camera" />
   </joint>

File: go2_navigation/xacro/gazebo.xacro (robot description, xacro)
@@ -13,5 +13,5 @@
             <frequency>10</frequency>
             <plot>
-                <link>base</link>
+                <link>base_link</link>
                 <pose>0 0 0 0 0 0</pose>
                 <material>Gazebo/Yellow</material>
@@ -120,5 +120,5 @@
         </visual>
     </gazebo>
-    <gazebo reference="base">
+    <gazebo reference="base_link">
         <turnGravityOff>false</turnGravityOff>
     </gazebo>

File: go2_navigation/xacro/robot.xacro (robot description, xacro)
@@ -17,8 +17,8 @@
             <origin rpy="0 0 0" xyz="0 0 0"/>
             <parent link="world"/>
-            <child link="base"/>
+            <child link="base_link"/>
         </joint>
     </xacro:if>
-    <link name="base">
+    <link name="base_link">
         <visual>
             <origin rpy="0 0 0" xyz="0 0 0"/>
@@ -30,5 +30,5 @@
     <joint name="floating_base" type="fixed">
         <origin rpy="0 0 0" xyz="0 0 0"/>
-        <parent link="base"/>
+        <parent link="base_link"/>
         <child link="trunk"/>
     </joint>
